File: boostlet.kicad_sch (KiCad schematic)
At the start: 52 parts, among them J1 Conn_01x13_Socket, J2 Conn_01x05_Socket, J3 Conn_01x05_Socket, Q1 BSS138, Q2 BSS138, U1 PAM2401, U2 AP2112K-3.3

Commit message: Version 1.2
Parts:
- removed C4: 680 uF @ 10 V, Capacitor_SMD:CP_Elec_10x10, symbol Device:C
- removed C6: 4.7 uF, Capacitor_SMD:C_1206_3216Metric_Pad1.33x1.80mm_HandSolder, symbol Device:C
- removed D1: D_Schottky 3A, Diode_SMD:D_SOD-123, symbol Device:D_Schottky
- removed J1: Conn_01x13_Socket, !EK_Library:Castellated_1x13_P2.54mm, symbol Connector:Conn_01x13_Socket
- removed J2, J3: Conn_01x05_Socket, !EK_Library:Castellated_1x05_P2.54mm, symbol Connector:Conn_01x05_Socket
- removed Q2: BSS138, Package_TO_SOT_SMD:SOT-23, symbol Transistor_FET:BSS138
- removed R4, R5: 10k, Resistor_SMD:R_1206_3216Metric_Pad1.30x1.75mm_HandSolder, symbol Device:R
- removed TP10, TP8, TP9: TestPoint, TestPoint:TestPoint_Pad_D1.5mm, symbol Connector:TestPoint
- removed U2: AP2112K-3.3, Package_TO_SOT_SMD:SOT-23-5, symbol Regulator_Linear:AP2112K-3.3
- added D2: PMEG40T30ERX 40V 3A, Diode_SMD:D_SOD-123, symbol Device:D_Schottky
- added J4: Conn_01x10_Socket, !RobotButterfly:Oval_1x10_P2.54mm, symbol Connector:Conn_01x10_Socket
- added Q3: DMG3415U, Package_TO_SOT_SMD:SOT-23, symbol Transistor_FET:DMG2301L
- added R11: 100k, Resistor_SMD:R_1206_3216Metric_Pad1.30x1.75mm_HandSolder, symbol Device:R
- added U4: AP2111H-3.3TRG1, Package_TO_SOT_SMD:SOT-223-3_TabPin2, symbol Regulator_Linear:AP1117-33
- C1: value 680 uF @ 10 V -> 1000 uF @ 16 V; Digikey 399-A765MN687M1ALAE013CT-ND -> 399-A768MS108M1CLAE015CT-ND; Digikey2 399-20537-1-ND -> (none)
- C2: Digikey 1276-1075-2-ND -> 1276-1075-1-ND
- C3: value 4.7 uF -> 1 uF; Digikey 1276-3181-1-ND -> 1276-3091-1-ND
- L1: value 2.2 uH, 3 A -> 4.7 uH, 3 A; footprint !EK_Library:INDUCTOR_IND_IFSC_1515AH_VIS-M -> Inductor_SMD:L_Taiyo-Yuden_NR-60xx_HandSoldering; Digikey 541-1404-1-ND -> SRN6045-4R7YCT-ND
- Q1: Digikey (none) -> 4530-BSS138CT-ND
- R1, R2: Digikey (none) -> RMCF1206FT10K0CT-ND
- R10: Digikey (none) -> 738-RMCF1206FT6K80CT-ND
- R9: Digikey (none) -> RMCF1206FG100RCT-ND
- renumbered C8 to C4, TP16 to TP15, TP15 to TP16
Connections:
- net 3.3V: now also J4.8 (Pin_8), U4.2 (VO)
- net 5V: now also F2.1, JP3.2 (B), J4.9 (Pin_9); no longer F2.2, JP3.1 (A)
- net BATT_SIG: now also J4.5 (Pin_5)
- net GND: now also J4.1 (Pin_1), J4.10 (Pin_10), R11.2, U4.1 (GND)
- net NEO_IN1: now also J4.7 (Pin_7)
- net NEO_OUT1: now also J4.6 (Pin_6)
- net VCC: now also J4.3 (Pin_3)
- net V_BATT: now also J4.4 (Pin_4)
- net at C3.1, JP2.2 (B), TP11.1: now also U4.3 (VI)
- net V_BOOST: now reaches C5.1, R7.1, TP12.1, U1.7 (OUT)
- net V_BOOST: now also C7.1, Q3.3 (D)
- new net: D2.1 (K), F2.2, JP3.1 (A), Q3.2 (S), TP14.1
- new net V_BUS: D2.2 (A), J4.2 (Pin_2), Q3.1 (G), R11.1
Other:
- note added: "AP2111H-3.3TRG1 outputs 3.3V 600 mA, max V_in = 6V"
- note added: "Boostlet! (C) Copyright Erin RobotZwrrl, Robot Missions Inc. 03-09-24 v1.2 RobotZwrrl.xyz/boostlet RobotMissions.org This hardware is released under: CERN Open Hardware License Version 2.0 - Permissive (CERN-OHL-P) Disclaimer: Distributed as is. No warranty is given. Not responsible or liable for any damage or harm that result from this product."
- note added: "Connector"
- note added: "Neopixel Level Shifter"
- note added: "Output Selector"
- note removed: "AP2114HA-3.3TRG1 outputs 3.3V 1A, max V_in = 6V"
- note removed: "Boostlet! (C) Copyright Erin RobotZwrrl, Robot Missions Inc. 12-30-23 v1.0 RobotZwrrl.xyz/boostlet RobotMissions.org This hardware is released under: CERN Open Hardware License Version 2.0 - Permissive (CERN-OHL-P) Disclaimer: Distributed as is. No warranty is given. Not responsible or liable for any damage or harm that result from this product."
- note removed: "Connectors"
- note removed: "Neopixel Level Shifters"
- moved on the sheet: C4, C7, F2, JP2, JP3, JP4, R10, R9, TP11, TP12, TP13, TP14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
