File: boostlet.kicad_sch (KiCad schematic)
At the start: 44 parts, among them J4 Conn_01x10_Socket, Q1 BSS138, Q3 DMG3415U, U1 PAM2401, U4 AP2111H-3.3TRG1

Commit message: Boostlet v1.2
Parts:
- removed JP2, JP4: SolderJumper_2_Open, Jumper:SolderJumper-2_P1.3mm_Open_RoundedPad1.0x1.5mm, symbol Jumper:SolderJumper_2_Open
- added JP2, JP4: SolderJumper_2_Bridged, Jumper:SolderJumper-2_P1.3mm_Bridged_RoundedPad1.0x1.5mm, symbol Jumper:SolderJumper_2_Bridged
Connections:
- net 3.3V: now also JP4.1 (A)
- net 5V: now also JP2.1 (A)
- net VCC: now also JP4.2 (B)
- net at C3.1, TP11.1, U4.3 (VI): now also JP2.2 (B)
Changed lines of the file:
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@@
 	)
 	(symbol
-		(lib_id "Jumper:SolderJumper_2_Open")
-		(at 170.18 148.59 0)
-		(unit 1)
-		(exclude_from_sim no)
-		(in_bom yes)
-		(on_board yes)
-		(dnp no)
-		(fields_autoplaced yes)
-		(property "Reference" "JP2"
-			(at 170.18 142.24 0)
-			(effects
-				(font
-					(size 1.27 1.27)
-				)
-			)
-		)
-		(property "Value" "SolderJumper_2_Open"
-			(at 170.18 144.78 0)
-			(effects
-				(font
-					(size 1.27 1.27)
-				)
-			)
-		)
-		(property "Footprint" "Jumper:SolderJumper-2_P1.3mm_Open_RoundedPad1.0x1.5mm"
-			(at 170.18 148.59 0)
-			(effects
-				(font
-					(size 1.27 1.27)
-				)
-				(hide yes)
-			)
-		)
-		(property "Datasheet" "~"
-			(at 170.18 148.59 0)
-			(effects
-				(font
-					(size 1.27 1.27)
-				)
-				(hide yes)
-			)
-		)
-		(property "Description" ""
-			(at 170.18 148.59 0)
-			(effects
-				(font
-					(size 1.27 1.27)
-				)
-				(hide yes)
-			)
-		)
-		(pin "1"
-		)
-		(pin "2"
-		)
-		(instances
-			(project "boostlet"
-				(path "/fed34468-19bb-4202-9cf6-96e1d57ad793"
-					(reference "JP2")
-					(unit 1)
-				)
-			)
-		)
-	)
-	(symbol
 		(lib_id "Device:C")
 		(at 179.07 162.56 0)
@@
 	)
 	(symbol
-		(lib_id "Jumper:SolderJumper_2_Open")
-		(at 245.11 148.59 0)
+		(lib_id "!EK_Library:PAM2401")
+		(at 113.03 55.88 0)
 		(unit 1)
 		(exclude_from_sim no)
@@
 		(dnp no)
 		(fields_autoplaced yes)
-		(property "Reference" "JP4"
-			(at 245.11 142.24 0)
+		(property "Reference" "U1"
+			(at 135.89 50.8 0)
 			(effects
 				(font
-					(size 1.27 1.27)
+					(size 1.524 1.524)
 				)
 			)
 		)
-		(property "Value" "SolderJumper_2_Open"
-			(at 245.11 144.78 0)
+		(property "Value" "PAM2401"
+			(at 135.89 53.34 0)
 			(effects
 				(font
-					(size 1.27 1.27)
+					(size 1.524 1.524)
 				)
 			)
 		)
-		(property "Footprint" "Jumper:SolderJumper-2_P1.3mm_Open_RoundedPad1.0x1.5mm"
-			(at 245.11 148.59 0)
+		(property "Footprint" "!EK_Library:PAM2401"
+			(at 113.03 81.28 0)
 			(effects
 				(font
 					(size 1.27 1.27)
+					(italic yes)
 				)
+				(justify left)
 				(hide yes)
 			)
 		)
-		(property "Datasheet" "~"
-			(at 245.11 148.59 0)
+		(property "Datasheet" "PAM2401SCADJ"
+			(at 113.03 78.74 0)
 			(effects
 				(font
 					(size 1.27 1.27)
+					(italic yes)
 				)
+				(justify left)
 				(hide yes)
 			)
 		)
 		(property "Description" ""
-			(at 245.11 148.59 0)
+			(at 113.03 55.88 0)
+			(effects
+				(font
+					(size 1.27 1.27)
+				)
+				(hide yes)
+			)
+		)
+		(property "Digikey" "PAM2401SCADJDICT-ND"
+			(at 124.46 85.09 0)
 			(effects
 				(font
@@
 		(pin "2"
 		)
+		(pin "3"
+		)
+		(pin "4"
+		)
+		(pin "5"
+		)
+		(pin "6"
+		)
+		(pin "7"
+		)
+		(pin "8"
+		)
 		(instances
 			(project "boostlet"
 				(path "/fed34468-19bb-4202-9cf6-96e1d57ad793"
-					(reference "JP4")
+					(reference "U1")
 					(unit 1)
 				)
@@
 	)
 	(symbol
-		(lib_id "!EK_Library:PAM2401")
-		(at 113.03 55.88 0)
+		(lib_id "Jumper:SolderJumper_2_Bridged")
+		(at 245.11 148.59 0)
 		(unit 1)
 		(exclude_from_sim no)
@@
 		(on_board yes)
 		(dnp no)
-		(fields_autoplaced yes)
-		(property "Reference" "U1"
-			(at 135.89 50.8 0)
-			(effects
-				(font
-					(size 1.524 1.524)
-				)
-			)
-		)
-		(property "Value" "PAM2401"
-			(at 135.89 53.34 0)
+		(property "Reference" "JP4"
+			(at 245.11 142.24 0)
 			(effects
 				(font
-					(size 1.524 1.524)
+					(size 1.27 1.27)
 				)
 			)
 		)
-		(property "Footprint" "!EK_Library:PAM2401"
-			(at 113.03 81.28 0)
+		(property "Value" "SolderJumper_2_Bridged"
+			(at 245.11 144.78 0)
 			(effects
 				(font
 					(size 1.27 1.27)
-					(italic yes)
 				)
-				(justify left)
-				(hide yes)
 			)
 		)
-		(property "Datasheet" "PAM2401SCADJ"
-			(at 113.03 78.74 0)
+		(property "Footprint" "Jumper:SolderJumper-2_P1.3mm_Bridged_RoundedPad1.0x1.5mm"
+			(at 245.11 148.59 0)
 			(effects
 				(font
 					(size 1.27 1.27)
-					(italic yes)
 				)
-				(justify left)
 				(hide yes)
 			)
 		)
-		(property "Description" ""
-			(at 113.03 55.88 0)
+		(property "Datasheet" "~"
+			(at 245.11 148.59 0)
 			(effects
 				(font
@@
 			)
 		)
-		(property "Digikey" "PAM2401SCADJDICT-ND"
-			(at 124.46 85.09 0)
+		(property "Description" "Solder Jumper, 2-pole, closed/bridged"
+			(at 245.11 148.59 0)
 			(effects
 				(font
@@
 		(pin "2"
 		)
-		(pin "3"
-		)
-		(pin "4"
-		)
-		(pin "5"
-		)
-		(pin "6"
-		)
-		(pin "7"
-		)
-		(pin "8"
-		)
 		(instances
 			(project "boostlet"
 				(path "/fed34468-19bb-4202-9cf6-96e1d57ad793"
-					(reference "U1")
+					(reference "JP4")
 					(unit 1)
 				)
@@
 					(unit 1)
 				)
+			)
+		)
+	)
+	(symbol
+		(lib_id "Jumper:SolderJumper_2_Bridged")
+		(at 170.18 148.59 0)
+		(unit 1)
+		(exclude_from_sim no)
+		(in_bom yes)
+		(on_board yes)
+		(dnp no)
+		(fields_autoplaced yes)
+		(property "Reference" "JP2"
+			(at 170.18 142.24 0)
+			(effects
+				(font
+					(size 1.27 1.27)
+				)
+			)
+		)
+		(property "Value" "SolderJumper_2_Bridged"
+			(at 170.18 144.78 0)
+			(effects
+				(font
+					(size 1.27 1.27)
+				)
+			)
+		)
+		(property "Footprint" "Jumper:SolderJumper-2_P1.3mm_Bridged_RoundedPad1.0x1.5mm"
+			(at 170.18 148.59 0)
+			(effects
+				(font
+					(size 1.27 1.27)
+				)
+				(hide yes)
+			)
+		)
+		(property "Datasheet" "~"
+			(at 170.18 148.59 0)
+			(effects
+				(font
+					(size 1.27 1.27)
+				)
+				(hide yes)
+			)
+		)
+		(property "Description" "Solder Jumper, 2-pole, closed/bridged"
+			(at 170.18 148.59 0)
+			(effects
+				(font
+					(size 1.27 1.27)
+				)
+				(hide yes)
+			)
+		)
+		(pin "1"
+		)
+		(pin "2"
+		)
+		(instances
+			(project "boostlet"
+				(path "/fed34468-19bb-4202-9cf6-96e1d57ad793"
+					(reference "JP2")
+					(unit 1)
+				)

Commit message: Mlep mlep rrrrr, zwap zwap zwap
Parts:
- C2: Digikey2 (none) -> 399-C1206C106K3PAC7800CT-ND
- R11, R3, R8: Digikey 311-100KFRCT-ND -> RMCF1206FT100KCT-ND; Digikey2 (none) -> 311-100KFRCT-ND
- R7: Digikey 311-750KFRCT-ND -> 738-RMCF1206FG750KCT-ND; Digikey2 (none) -> 311-750KFRCT-ND
Other:
- note added: "Boostlet! (C) Copyright Erin RobotZwrrl, Robot Missions Inc. 04-09-24 v1.3 RobotZwrrl.xyz/boostlet RobotMissions.org This hardware is released under: CERN Open Hardware License Version 2.0 - Permissive (CERN-OHL-P) Disclaimer: Distributed as is. No warranty is given. Not responsible or liable for any damage or harm that result from this product."
- note removed: "Boostlet! (C) Copyright Erin RobotZwrrl, Robot Missions Inc. 03-09-24 v1.2 RobotZwrrl.xyz/boostlet RobotMissions.org This hardware is released under: CERN Open Hardware License Version 2.0 - Permissive (CERN-OHL-P) Disclaimer: Distributed as is. No warranty is given. Not responsible or liable for any damage or harm that result from this product."
Changed lines of the file:
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@@
 		)
 	)
-	(text "Boostlet! (C) Copyright Erin RobotZwrrl, Robot Missions Inc.\n03-09-24 v1.2\nRobotZwrrl.xyz/boostlet\nRobotMissions.org\n\nThis hardware is released under:\nCERN Open Hardware License Version 2.0 - Permissive (CERN-OHL-P)\n\nDisclaimer: Distributed as is. No warranty is given. Not responsible \nor liable for any damage or harm that result from this product."
+	(text "Boostlet! (C) Copyright Erin RobotZwrrl, Robot Missions Inc.\n04-09-24 v1.3\nRobotZwrrl.xyz/boostlet\nRobotMissions.org\n\nThis hardware is released under:\nCERN Open Hardware License Version 2.0 - Permissive (CERN-OHL-P)\n\nDisclaimer: Distributed as is. No warranty is given. Not responsible \nor liable for any damage or harm that result from this product."
 		(exclude_from_sim no)
 		(at 300.99 264.16 0)
@@
 			)
 		)
-		(property "Digikey" "311-750KFRCT-ND"
+		(property "Digikey" "738-RMCF1206FG750KCT-ND"
+			(at 193.04 71.12 0)
+			(effects
+				(font
+					(size 1.27 1.27)
+				)
+				(hide yes)
+			)
+		)
+		(property "Digikey2" "311-750KFRCT-ND"
 			(at 193.04 71.12 0)
 			(effects
@@
 			)
 		)
+		(property "Digikey2" "399-C1206C106K3PAC7800CT-ND"
+			(at 90.17 78.74 0)
+			(effects
+				(font
+					(size 1.27 1.27)
+				)
+				(hide yes)
+			)
+		)
 		(pin "1"
 		)
@@
 			)
 		)
-		(property "Digikey" "311-100KFRCT-ND"
+		(property "Digikey" "RMCF1206FT100KCT-ND"
+			(at 266.7 86.36 0)
+			(effects
+				(font
+					(size 1.27 1.27)
+				)
+				(hide yes)
+			)
+		)
+		(property "Digikey2" "311-100KFRCT-ND"
 			(at 266.7 86.36 0)
 			(effects
@@
 			)
 		)
-		(property "Digikey" "311-100KFRCT-ND"
+		(property "Digikey" "RMCF1206FT100KCT-ND"
+			(at 193.04 85.09 0)
+			(effects
+				(font
+					(size 1.27 1.27)
+				)
+				(hide yes)
+			)
+		)
+		(property "Digikey2" "311-100KFRCT-ND"
 			(at 193.04 85.09 0)
 			(effects
@@
 			)
 		)
-		(property "Digikey" "311-100KFRCT-ND"
+		(property "Digikey" "RMCF1206FT100KCT-ND"
 			(at 66.04 63.5 0)
 			(effects
 				(font
+					(size 1.27 1.27)
+				)
+				(hide yes)
+			)
+		)
+		(property "Digikey2" "311-100KFRCT-ND"
+			(at 66.04 63.5 90)
+			(effects
+				(font
