File: archive/v1.0/boostlet.kicad_sch (KiCad schematic)
At the start: 52 parts, among them J1 Conn_01x13_Socket, J2 Conn_01x05_Socket, J3 Conn_01x05_Socket, Q1 BSS138, Q2 BSS138, U1 PAM2401, U2 AP2112K-3.3

Commit message: Mysterious vault of boostletland
Parts:
- C2: Digikey 1276-1075-2-ND -> 1276-1075-1-ND
- Q1, Q2: Digikey (none) -> 4530-BSS138CT-ND
- R1, R2, R4, R5: Digikey (none) -> RMCF1206FT10K0CT-ND
- R10: Digikey (none) -> 738-RMCF1206FT6K80CT-ND
- R9: Digikey (none) -> RMCF1206FG100RCT-ND
- U2: Digikey (none) -> AP2112K-3.3TRG1DICT-ND
Changed lines of the file:
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@@
+      (effects (font (size 1.27 1.27)) hide)
+    )
+    (property "Digikey" "RMCF1206FT10K0CT-ND" (at 184.15 246.38 0)
       (effects (font (size 1.27 1.27)) hide)
     )
@@
       (effects (font (size 1.27 1.27)) (justify left) hide)
     )
+    (property "Digikey" "4530-BSS138CT-ND" (at 66.04 254 90)
+      (effects (font (size 1.27 1.27)) hide)
+    )
     (pin "1")
     (pin "2")
@@
       (effects (font (size 1.27 1.27)) hide)
     )
+    (property "Digikey" "RMCF1206FG100RCT-ND" (at 316.23 60.96 0)
+      (effects (font (size 1.27 1.27)) hide)
+    )
     (pin "1")
     (pin "2")
@@
     )
     (property "Datasheet" "~" (at 50.8 245.11 0)
+      (effects (font (size 1.27 1.27)) hide)
+    )
+    (property "Digikey" "RMCF1206FT10K0CT-ND" (at 50.8 245.11 0)
       (effects (font (size 1.27 1.27)) hide)
     )
@@
       (effects (font (size 1.27 1.27)) hide)
     )
-    (property "Digikey" "1276-1075-2-ND" (at 90.17 78.74 0)
+    (property "Digikey" "1276-1075-1-ND" (at 90.17 78.74 0)
       (effects (font (size 1.27 1.27)) hide)
     )
@@
     )
     (property "Datasheet" "https://www.diodes.com/assets/Datasheets/AP2112.pdf" (at 248.92 152.4 0)
+      (effects (font (size 1.27 1.27)) hide)
+    )
+    (property "Digikey" "AP2112K-3.3TRG1DICT-ND" (at 248.92 154.94 0)
       (effects (font (size 1.27 1.27)) hide)
     )
@@
       (effects (font (size 1.27 1.27)) hide)
     )
+    (property "Digikey" "RMCF1206FT10K0CT-ND" (at 157.48 246.38 0)
+      (effects (font (size 1.27 1.27)) hide)
+    )
     (pin "1")
     (pin "2")
@@
     (property "Datasheet" "https://www.onsemi.com/pub/Collateral/BSS138-D.PDF" (at 172.72 255.27 0)
       (effects (font (size 1.27 1.27)) (justify left) hide)
+    )
+    (property "Digikey" "4530-BSS138CT-ND" (at 172.72 255.27 90)
+      (effects (font (size 1.27 1.27)) hide)
     )
     (pin "1")
@@
       (effects (font (size 1.27 1.27)) hide)
     )
+    (property "Digikey" "738-RMCF1206FT6K80CT-ND" (at 316.23 76.2 0)
+      (effects (font (size 1.27 1.27)) hide)
+    )
     (pin "1")
     (pin "2")
@@
       (effects (font (size 1.27 1.27)) hide)
     )
+    (property "Digikey" "RMCF1206FT10K0CT-ND" (at 77.47 245.11 0)
+      (effects (font (size 1.27 1.27)) hide)
+    )
